File: Pcb/Display/Display.brd (EAGLE design)
At the start: 63.5 x 76.4 mm, 31 parts, among them J2 47219-2001, Q1 310mA/60V/1.6Ω

Commit message: Updated PCB files and ported some of the graphics functions. The graphics changes are not tested yet.
Parts:
- added R14: 10, adafruit:R0805
- added R15: 1k, adafruit:R0805
- added TP1: TPTP09R, testpad:TP09R
- moved Q1 0.89 mm to (4.19, 36.2)
- moved J2 0.10 mm to (49.7, 21.9), flipped to the bottom, turned to 90 degrees
Connections:
- new net N$4: R15.2, TFT2.46
- new net RST: R14.2, TFT2.10, TFT2.47, TP1.TP
- net GND: no longer TFT2.47
- net I2C_INT: now also R15.1; no longer TFT2.46
- net RDX: now also TFT2.35; no longer TFT2.36
- net VCC: now also R14.1
- net WRX: now also TFT2.36; no longer TFT2.35
Routing:
- net GND: track 257.9 -> 198.2 mm, vias 3 -> 5
- net RST: track 0.00 -> 44.2 mm, vias 0 -> 1
- net SD_DAT0: track 14.1 -> 25.7 mm
- net I2C_INT: track 54.0 -> 46.0 mm
- net R13: track 64.7 -> 57.8 mm
- net N$4: track 0.00 -> 6.09 mm
- net N$6: track 39.4 -> 34.5 mm
- net VCC: track 183.8 -> 179.0 mm, vias 5 -> 6
- net R12: track 26.7 -> 22.6 mm
- net N$7: track 38.4 -> 34.4 mm
- net N$9: track 37.4 -> 34.4 mm
- net SD_CLK: track 14.0 -> 16.4 mm
- net N$8: track 36.5 -> 34.6 mm
- net WRX: track 37.6 -> 36.2 mm
- net RDX: track 36.6 -> 35.6 mm
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