File: Pcb/Main/Main_v3.sch (EAGLE design)
At the start: 60 parts, among them IC1 CC3220MODASF12MONR, J1 CORTEX_JTAG_DEBUG_PTH, J5 MOLEX_43045-0200MOLEX_43045-0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, Q1 220mA/50V/3.5Ω, U1 AD7993BRU-0, U2 LTC3440EMSPBF, U3 MAX17201G+T

Commit message: Updated PCB files and ported some of the graphics functions. The graphics changes are not tested yet.
Parts:
- added 74LVC: SOP65P400X110-8N, SOP65P400X110-8N:SOP65P400X110-8N
- added D2, D7: (no value), adafruit:DIODESOD-323F
- added R13: 10k, rcl:R-US_R0805
- added R14: 1k, rcl:R-US_R0805
- R6: value (none) -> 10k
- renumbered U$1 to MCP, U2 to LTC, U3 to MAX
Connections:
- new net I2C_ADC: 74LVC.1A, R14.1
- new net I2C_DSP: 74LVC.3A, JP2.3
- new net I2C_MAX: 74LVC.2A, R20.2
- new net N$10: IC1.ANT_SEL1
- new net N$11: IC1.ANT_SEL2
- new net N$12: IC1.NC_2
- new net N$13: IC1.RF_BG
- new net N$14: IC1.FLASH_SPI_MOSI
- new net N$15: IC1.FLASH_SPI_CLK
- new net N$16: IC1.FLASH_SPI_NCS_IN
- new net N$17: IC1.FLASH_SPI_MISO
- new net N$18: IC1.NC_1
- new net N$3: IC1.NC_5
- new net N$4: R14.2, U1.ALERT/BUSY
- new net N$5: IC1.GPIO30
- new net N$6: IC1.NC_4
- new net N$7: IC1.VBAT_RESET
- new net N$8: IC1.NC_3
- new net N$9: IC1.NC_6
- net GND: now also 74LVC.GND, D2.A, U$2.1, U$2.12, U$2.13, U$2.16, U$2.4, U$2.5, U$2.8, U$2.9; no longer U$2.10, U$2.11, U$2.14, U$2.15, U$2.2, U$2.3, U$2.6, U$2.7
- net I2C_INT: now also 74LVC.1Y, 74LVC.2Y, 74LVC.3Y, R13.2; no longer JP2.3, R20.2, U1.ALERT/BUSY
- net LTC_IND1: now also D2.C
- net LTC_IND2: now also D7.A
- net VCC: now also 74LVC.VCC, D7.C, R13.1, U$2.10, U$2.14, U$2.2, U$2.6; no longer U$2.12, U$2.16, U$2.4, U$2.8
- net VIN1: now also U$2.15; no longer U$2.13
- net VIN2: now also U$2.7; no longer U$2.5
- net VIN3: now also U$2.11; no longer U$2.9
- net VIN4: now also U$2.3; no longer U$2.1
